File: vg.kicad_pcb (KiCad board)
At the start: 4 copper layers, 36 x 36 mm, 45 parts, among them J1 Conn_01x07, J2 Conn_01x08, J3 Conn_01x03, Q1 2N7002, Q3 SI2301CDS-T1-GE3, U1 TPS62203DBV, U2 IRLML6344TRPBF, U3 STM32L072CBTx, Y1 32768Hz - 12,5 pF

Commit message: add 2nd pin row
Parts:
- added J4: Conn_01x07, Connector_PinHeader_2.54mm:PinHeader_1x07_P2.54mm_Vertical, F.Cu at (109.1, 51.7)
- J2: footprint Connector_PinHeader_2.54mm:PinHeader_1x08_P2.54mm_Horizontal -> Connector_PinHeader_2.54mm:PinHeader_1x08_P2.54mm_Vertical
- moved L1 1.74 mm to (112.5, 58.0)
- moved J2 1.35 mm to (109.1, 55.4)
Routing:
- net SCREEN_DIN: track 7.57 -> 18.4 mm, vias 2 -> 1
- net SCREEN_DC: track 13.9 -> 24.2 mm
- net SCREEN_CS: track 7.84 -> 16.3 mm
- net SCREEN_RES: track 9.05 -> 14.4 mm
- net SCREEN_CLK: track 5.72 -> 10.9 mm
- net +3V3: track 32.6 -> 31.0 mm, vias 13 -> 15
- net GND: vias 27 -> 29
Other:
- board text added: "J2 - adafruit display J4 - generic"

Commit message: dont pour all the way to the edge; replace speaker series cap with 0805 for better thermal; gnd vias on both sides of islands; long trace series resistors close to chip; shorter filter cap connections
Parts:
- added R14: 330, Resistor_SMD:R_0402_1005Metric, F.Cu at (131.0, 70.0)
- added R15: 330, Resistor_SMD:R_0402_1005Metric, F.Cu at (131.0, 68.9)
- added R7: 330, Resistor_SMD:R_0402_1005Metric, F.Cu at (134.3, 77.3)
- added R8: 330, Resistor_SMD:R_0402_1005Metric, F.Cu at (131.1, 72.5)
- R10: footprint Resistor_SMD:R_0402_1005Metric -> PCM_JLCPCB:R_0402
- R9: footprint Resistor_SMD:R_0402_1005Metric -> PCM_JLCPCB:R_0805
- moved R12 20.2 mm to (129.3, 61.2), turned to 180 degrees
- moved R13 20.1 mm to (115.3, 64.3)
- moved R2 16.9 mm to (122.3, 70.4), turned to -90 degrees
- moved R11 10.6 mm to (119.5, 71.8), turned to 90 degrees
- moved R10 6.08 mm to (111.5, 76.1), turned to 180 degrees
- moved JP1 2.59 mm to (104.5, 77.5), turned to -90 degrees
- moved R5 1.57 mm to (119.8, 82.0), turned to -90 degrees
- moved R4 1.44 mm to (111.7, 81.9), turned to -90 degrees
- moved R9 0.92 mm to (117.8, 75.1)
- moved R6 0.35 mm to (128.6, 80.8)
- moved Y1 0.31 mm to (129.1, 65.8)
- moved C2 0.31 mm to (130.8, 66.7)
- moved C3 0.31 mm to (130.8, 64.7)
- moved C4 0.13 mm to (128.7, 62.9), turned to -90 degrees
Connections:
- J1 pad 4: SWCLK -> Net-(J1-Pin_4)
- J1 pad 5: SWDIO -> Net-(J1-Pin_5)
- J1 pad 6: USART1_RX -> Net-(J1-Pin_6)
- J1 pad 7: USART1_TX -> Net-(J1-Pin_7)
Routing:
- net Net-(R12-Pad1): track 3.56 -> 35.1 mm, vias 0 -> 4
- net RIGHT_BTN: track 38.4 -> 8.98 mm, vias 8 -> 2
- net MIDDLE_BTN: track 31.5 -> 2.43 mm, vias 4 -> 0
- net Net-(R13-Pad1): track 3.36 -> 30.2 mm, vias 0 -> 4
- net Net-(R11-Pad1): track 3.47 -> 18.9 mm, vias 0 -> 2
- net LEFT_BTN: track 17.7 -> 3.84 mm, vias 2 -> 0
- net VBATT_ANA: track 30.1 -> 42.4 mm
- net GND: track 4.72 -> 10.7 mm, vias 29 -> 54
- net +3V3: track 31.0 -> 35.6 mm, vias 15 -> 12
- net SWDIO: track 24.1 -> 20.5 mm
- net SWCLK: track 17.3 -> 14.1 mm
- net Net-(J1-Pin_4): track 0.00 -> 3.13 mm
- net USART1_RX: track 28.8 -> 25.8 mm
- net Net-(J1-Pin_5): track 0.00 -> 2.55 mm
- net BOOT0: track 28.8 -> 26.3 mm
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- added copper zone on B.Cu, net GND

Commit message: fix some LCSC #s
Routing:
- net GND: vias 54 -> 58
Changed lines of the file:
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@@
 		)
 		(fp_text user "${REFERENCE}"
-			(at 0 7.62 360)
+			(at 0 7.62 0)
 			(layer "F.Fab")
 			(effects
@@
 		(tags "resistor")
 		(property "Reference" "R10"
-			(at -1.05 -0.85 360)
+			(at -1.05 -0.85 0)
 			(layer "F.SilkS")
 			(hide yes)
@@
 		)
 		(property "Value" "1k"
-			(at 0 0.2 360)
+			(at 0 0.2 0)
 			(layer "F.Fab")
 			(hide yes)
@@
 		)
 		(fp_text user "${REFERENCE}"
-			(at 0 -0.25 360)
+			(at 0 -0.25 0)
 			(layer "F.Fab")
 			(hide yes)
@@
 		)
 		(fp_text user "${REFERENCE}"
-			(at 0 1.27 360)
+			(at 0 1.27 0)
 			(layer "F.Fab")
 			(effects
@@
 		(tags "resistor")
 		(property "Reference" "R7"
-			(at 0 -1.17 360)
+			(at 0 -1.17 0)
 			(layer "F.SilkS")
 			(hide yes)
@@
 		)
 		(property "Value" "330"
-			(at 0 1.17 360)
+			(at 0 1.17 0)
 			(layer "F.Fab")
 			(effects
@@
 		)
 		(fp_text user "${REFERENCE}"
-			(at 0 0 360)
+			(at 0 0 0)
 			(layer "F.Fab")
 			(effects
@@
 		(tags "resistor")
 		(property "Reference" "R12"
-			(at 0 -1.17 360)
+			(at 0 -1.17 0)
 			(layer "F.SilkS")
 			(hide yes)
@@
 		)
 		(property "Value" "330"
-			(at 0 1.17 360)
+			(at 0 1.17 0)
 			(layer "F.Fab")
 			(effects
@@
 		)
 		(fp_text user "${REFERENCE}"
-			(at 0 0 360)
+			(at 0 0 0)
 			(layer "F.Fab")
 			(effects
@@
 	)
 	(via
+		(at 117.075 61.575)
+		(size 0.4)
+		(drill 0.2)
+		(layers "F.Cu" "B.Cu")
+		(free yes)
+		(net 2)
+	)
+	(via
 		(at 131.25 71.55)
 		(size 0.4)
@@
 	)
 	(via
+		(at 114.475 64.275)
+		(size 0.4)
+		(drill 0.2)
+		(layers "F.Cu" "B.Cu")
+		(free yes)
+		(net 2)
+	)
+	(via
 		(at 120.45 75.9)
 		(size 0.4)
@@
 	)
 	(via
+		(at 123.475 76.925)
+		(size 0.4)
+		(drill 0.2)
+		(layers "F.Cu" "B.Cu")
+		(free yes)
+		(net 2)
+	)
+	(via
 		(at 129.05 77.2)
 		(size 0.4)
@@
 		(size 0.4)
 		(drill 0.2)
+		(layers "F.Cu" "B.Cu")
+		(free yes)
+		(net 2)
+	)
+	(via
+		(at 113.775 59.525)
+		(size 0.4)
+		(drill 0.2)
